File: Circuits/TestStand/TestStand.kicad_sch (KiCad schematic)
At the start: 109 parts, among them IC1 STP85NF55, J1 2601-1107, J10 Screw_Terminal_01x03, J11 Screw_Terminal_01x03, J12 Screw_Terminal_01x03, J13 Screw_Terminal_01x03, J14 CONN4_2606-1104/010-000_WAG, J15 Conn_Coaxial, J18 2601-1107, J2 2601-1107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

Commit message: whatever I was working on last night
Parts:
- added J16: CONN4_2606-1104/010-000_WAG, Library:2606-1104&slash_010-000, symbol 2024-08-14_06-49-46:CONN4_2606-1104/010-000_WAG
Connections:
- net GND: now also J16.4

Commit message: added optoisolators and did some routing
Parts:
- removed J16: CONN4_2606-1104/010-000_WAG, Library:2606-1104&slash_010-000, symbol 2024-08-14_06-49-46:CONN4_2606-1104/010-000_WAG
- added J17: Screw_Terminal_01x03, Library:CONN3_2601-1103_WAG, symbol 2024-08-14_06-29-14:2601-1103
- added R21, R22, R23: 220, Resistor_SMD:R_0805_2012Metric, symbol Device:R_US
- added U10, U11, U9: VO615A-X001, DIP-4_VO615A_VIS, symbol 2024-08-16_03-45-33:VO615A-X001
Connections:
- net +BATT: now also U10.4 (C), U11.4 (C), U9.4 (C)
- net GND: now also J3.5 (3_1), J3.6 (3_2), R21.1, R22.1, R23.1
- net GPIN: now reaches U4.43 (21_A7_RX5_BCLK1)
- net GPIN: now also U11.1 (A)
- net YPIN: now reaches U4.44 (22_A8_CTX1)
- net YPIN: now also U10.1 (A)
- net RPIN: now reaches U4.45 (23_A9_CRX1_MCLK1)
- net RPIN: now also U9.1 (A)
- new net: R22.2, U10.2 (C)
- new net: R23.2, U9.2 (C)
- new net: R21.2, U11.2 (C)
- new net GREEN: J17.5 (3_1), J17.6 (3_2), U11.3 (E)
- new net RED: J17.1 (1_1), J17.2 (1_2), U9.3 (E)
- new net YELLOW: J17.3 (2_1), J17.4 (2_2), U10.3 (E)
- no-connect marks 44 -> 39
Other:
- note added: "GND For LEDS"
